File: 5sec_challenge_display/5sec_challenge_display.kicad_pcb (KiCad board)
At the start: 2 copper layers, 66 x 50.8 mm, 5 parts, among them J1 Conn_01x09_Socket, J2 Conn_01x09_Socket, J3 Conn_01x15_Socket, J4 Conn_01x15_Socket, J5 Conn_01x07_Pin

Commit message: 修正
Parts:
- J5: footprint Connector_PinHeader_2.54mm:PinHeader_1x07_P2.54mm_Vertical -> Connector_PinHeader_2.54mm:PinHeader_1x07_P2.54mm_Horizontal
- moved J5 12.7 mm to (139.7, 111.8), turned to -90 degrees
Connections:
- J5 pad 1: +5V -> GND
- J5 pad 2: +5V -> GND
- J5 pad 3: /DIN -> /LATCH
- J5 pad 5: /LATCH -> /DIN
- J5 pad 6: GND -> +5V
- J5 pad 7: GND -> +5V
Routing:
- net /CLK: track 29.6 -> 27.1 mm
- net /DIN: track 29.6 -> 27.1 mm
- net /LATCH: track 82.5 -> 80.0 mm
Other:
- board size 66 x 50.8 mm -> 66 x 52.3 mm

Commit message: 修正
Parts:
- J1, J2: footprint Connector_PinHeader_2.54mm:PinHeader_1x09_P2.54mm_Vertical -> Connector_PinSocket_2.54mm:PinSocket_1x09_P2.54mm_Vertical
- J3, J4: footprint Connector_PinHeader_2.54mm:PinHeader_1x15_P2.54mm_Vertical -> Connector_PinSocket_2.54mm:PinSocket_1x15_P2.54mm_Vertical
Other:
- outline, holes or cut-outs redrawn
