File: 5sec_challenge_display/5sec_challenge_display.kicad_sch (KiCad schematic)
At the start: 5 parts, among them J1 Conn_01x09_Socket, J2 Conn_01x09_Socket, J3 Conn_01x15_Socket, J4 Conn_01x15_Socket, J5 Conn_01x07_Pin

Commit message: 修正
Parts:
- J5: footprint Connector_PinHeader_2.54mm:PinHeader_1x07_P2.54mm_Vertical -> Connector_PinHeader_2.54mm:PinHeader_1x07_P2.54mm_Horizontal
Connections:
- net +5V: now also J5.6 (Pin_6), J5.7 (Pin_7); no longer J5.1 (Pin_1), J5.2 (Pin_2)
- net DIN: now also J5.5 (Pin_5); no longer J5.3 (Pin_3)
- net GND: now also J5.1 (Pin_1), J5.2 (Pin_2); no longer J5.6 (Pin_6), J5.7 (Pin_7)
- net LATCH: now also J5.3 (Pin_3); no longer J5.5 (Pin_5)
Other:
- moved on the sheet: J5
Changed lines of the file:
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@@
 	(symbol
 		(lib_id "Connector:Conn_01x07_Pin")
-		(at 110.49 113.03 90)
+		(at 110.49 113.03 270)
+		(mirror x)
 		(unit 1)
 		(exclude_from_sim no)
@@
 		(on_board yes)
 		(dnp no)
-		(fields_autoplaced yes)
 		(property "Reference" "J5"
 			(at 110.49 115.57 90)
@@
 			)
 		)
-		(property "Footprint" "Connector_PinHeader_2.54mm:PinHeader_1x07_P2.54mm_Vertical"
+		(property "Footprint" "Connector_PinHeader_2.54mm:PinHeader_1x07_P2.54mm_Horizontal"
 			(at 110.49 113.03 0)
 			(effects

Commit message: 修正
Parts:
- J1, J2: footprint Connector_PinHeader_2.54mm:PinHeader_1x09_P2.54mm_Vertical -> Connector_PinSocket_2.54mm:PinSocket_1x09_P2.54mm_Vertical
- J3, J4: footprint Connector_PinHeader_2.54mm:PinHeader_1x15_P2.54mm_Vertical -> Connector_PinSocket_2.54mm:PinSocket_1x15_P2.54mm_Vertical
Changed lines of the file:
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@@
 			)
 		)
-		(property "Footprint" "Connector_PinHeader_2.54mm:PinHeader_1x09_P2.54mm_Vertical"
+		(property "Footprint" "Connector_PinSocket_2.54mm:PinSocket_1x09_P2.54mm_Vertical"
 			(at 88.9 55.88 0)
 			(effects
@@
 			)
 		)
-		(property "Footprint" "Connector_PinHeader_2.54mm:PinHeader_1x15_P2.54mm_Vertical"
+		(property "Footprint" "Connector_PinSocket_2.54mm:PinSocket_1x15_P2.54mm_Vertical"
 			(at 120.65 55.88 0)
 			(effects
@@
 			)
 		)
-		(property "Footprint" "Connector_PinHeader_2.54mm:PinHeader_1x15_P2.54mm_Vertical"
+		(property "Footprint" "Connector_PinSocket_2.54mm:PinSocket_1x15_P2.54mm_Vertical"
 			(at 120.65 71.12 0)
 			(effects
@@
 			)
 		)
-		(property "Footprint" "Connector_PinHeader_2.54mm:PinHeader_1x09_P2.54mm_Vertical"
+		(property "Footprint" "Connector_PinSocket_2.54mm:PinSocket_1x09_P2.54mm_Vertical"
 			(at 88.9 71.12 0)
 			(effects
