File: 5sec_challenge_mother/5sec_challenge_mother.kicad_pcb (KiCad board)
At the start: 2 copper layers, 66 x 33.7 mm, 7 parts, among them J1 Conn_01x07_Socket, J2 Barrel_Jack_Switch, U1 L7805

Commit message: スイッチ追加
Parts:
- added J3: Conn_01x02, Connector_JST:JST_XH_B2B-XH-AM_1x02_P2.50mm_Vertical, F.Cu at (134.6, 109.2)
- added SW1: SW_Push, Button_Switch_THT:SW_PUSH_6mm, F.Cu at (155.7, 111.5)
Connections:
- A1 pad 22: unconnected-(A1-A3-Pad22) -> Net-(A1-A3)
Routing:
- net Net-(A1-A3): track 0.00 -> 24.5 mm
Other:
- board size 66 x 33.7 mm -> 66 x 42.5 mm
